File: lisalite/lisalite.kicad_pcb (KiCad board)
At the start: 2 copper layers, 103.7 x 65 mm, 16 parts, among them J1 LisaLite FDD Connector, J2 LisaLite Twiggy Port Connector, U1 5MHz XTAL, U2 74LS74, U3 74LS393, U4 74LS85, U5 74LS85, U6 74LS164

Commit message: final commit for rev 1.0
Parts:
- added G***: LOGO, LOGO, F.Cu at (59.4, 73.3)
- added G***: LOGO, LOGO, F.Cu at (110.5, 85.7)
- moved C1 33.1 mm to (66.7, 58.0)
- moved C2 33.1 mm to (66.7, 31.3)
- moved C5 33.1 mm to (104.8, 31.3)
- moved C6 33.1 mm to (117.5, 31.3)
- moved U1 33.1 mm to (67.9, 63.0)
- moved U2 33.1 mm to (67.9, 36.3)
- moved U3 33.1 mm to (80.6, 36.3)
- moved U5 33.1 mm to (106.0, 36.3)
- moved C3 33.1 mm to (79.4, 31.3)
- moved C4 33.1 mm to (92.1, 31.3)
- moved J1 33.1 mm to (115.6, 64.1)
- moved J2 33.1 mm to (147.3, 48.9)
- moved R1 33.1 mm to (131.4, 31.3)
- moved C7 33.1 mm to (139.9, 46.3)
- moved U4 33.1 mm to (93.3, 36.3)
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Connections:
- J2 pad 25: +5V -> unconnected-(J2-+5V-Pad25)
- U2 pad 14: (no net) -> +5V
- U2 pad 7: (no net) -> GND
Routing:
- net +5V: track 0.00 -> 299.5 mm
- net +12V: track 0.00 -> 186.5 mm
- net Net-(J1-RD): track 0.00 -> 92.6 mm
- net Net-(J1-WRTDATA): track 0.00 -> 91.0 mm
- net Net-(U2A-~{R}): track 0.00 -> 90.8 mm
- net Net-(J1-CA0): track 0.00 -> 81.8 mm
- net Net-(J1-ENBL): track 0.00 -> 75.5 mm
- net Net-(U1-OUT): track 0.00 -> 63.6 mm
- net Net-(U2A-D): track 0.00 -> 55.9 mm, vias 0 -> 1
- net Net-(U3B-Q3): track 0.00 -> 55.6 mm
- net Net-(J1-WRTGATE): track 0.00 -> 51.5 mm
- net Net-(J1-SEL): track 0.00 -> 51.3 mm
- net Net-(J1-LSTRB): track 0.00 -> 50.6 mm
- net Net-(J1-CA2): track 0.00 -> 48.7 mm
- net Net-(J2-MOTRCLK): track 0.00 -> 47.4 mm, vias 0 -> 1
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- added copper zone on B.Cu, net GND
- added copper zone on F.Cu, net GND
Other:
- outline, holes or cut-outs redrawn
- board text added: "149"
- board text added: "620 -"
- board text added: "820-4043-A"
- board text added: "LITE ADAPTER"
- board text added: "LS164"
- board text added: "LS393"
- board text added: "LS74"
- board text added: "LS85"
- board text added: "OSC"
- board text added: "© 1983"
