File: lisalite/lisalite.kicad_sch (KiCad schematic)
At the start: 4 parts, among them U1 74LS85, U2 74LS393, U3 74LS85, U4 74LS74

Commit message: schematic updates
Parts:
- added R1: 3.3K, symbol Device:R_US
- added U6: 74LS164, Package_DIP:DIP-14_W7.62mm, symbol 74xx_Custom:74LS164
- added X1: TFT680, Crystal:Crystal_AT310_D3.0mm_L10.0mm_Horizontal, symbol Oscillator:TFT680
- renumbered U4 to U2, U2 to U3, U3 to U4, U1 to U5
Connections:
- net at U3.1 (CP): now also U2.3 (C), X1.8 (OUT)
- net GND: now reaches U3.2 (MR)
- net GND: now also U3.12 (MR), U4.2 (Ia<b), U4.3 (Ia=b), U4.4 (Ia>b), U4.8 (GND), U6.7 (GND), X1.7 (GND)
- net at U3.3 (Q0): now also U4.9 (B0)
- net at U3.4 (Q1): now also U4.11 (B1)
- net at U3.5 (Q2): now also U4.14 (B2)
- net at U3.6 (Q3): now also U3.13 (CP), U4.1 (B3)
- net at U5.1 (B3): now also U3.8 (Q3)
- net at U5.10 (A0): now also U6.10 (Qe)
- net at U5.11 (B1): now also U3.10 (Q1)
- net at U5.12 (A1): now also U6.11 (Qf)
- net at U5.13 (A2): now also U6.12 (Qg)
- net at U5.14 (B2): now also U3.9 (Q2)
- net at U5.15 (A3): now also U6.13 (Qh)
- net at U5.2 (Ia<b): now also U4.7 (Oa<b)
- net at U5.3 (Ia=b): now also U4.6 (Oa=b)
- net at U5.4 (Ia>b): now also U4.5 (Oa>b)
- net at U5.7 (Oa<b): now also U2.2 (D)
- net at U5.9 (B0): now also U3.11 (Q0)
- net at U4.10 (A0): now also U6.3 (Qa)
- net at U4.12 (A1): now also U6.4 (Qb)
- net at U4.13 (A2): now also U6.5 (Qc)
- net at U4.15 (A3): now also U6.6 (Qd)
- net at U2.1 (~{R}): now also U2.4 (~{S}), R1.2, U6.9 (/CLR)
- new net +5V: R1.1, U6.14 (VCC), X1.14 (Vcc)
- no-connect marks 0 -> 4
Other:
- moved on the sheet: U2A, U2B, U2C, U3A, U3B, U4, U4C, U5

Commit message: generated pcb
Parts:
- removed unit 3 of U4
- added C1, C2, C3, C4, C5, C6: 0.1uF 50V, Capacitor_THT:C_Axial_L3.8mm_D2.6mm_P10.00mm_Horizontal, symbol Device:C
- added C7: 10uF 16V, Capacitor_THT:CP_Axial_L10.0mm_D6.0mm_P15.00mm_Horizontal, symbol Device:C_Polarized_US
- added J1: LisaLite FDD Connector, Connector_PinHeader_2.54mm:PinHeader_2x10_P2.54mm_Vertical, symbol Connector_Custom:Apple_Lisa_LisaLite_FDD_Connector
- added J2: LisaLite Twiggy Port Connector, Connector_PinHeader_2.54mm:PinHeader_2x13_P2.54mm_Vertical, symbol Connector_Custom:Apple_Lisa_LisaLite_Twiggy_Connector
- R1: footprint (none) -> Resistor_THT:R_Axial_DIN0309_L9.0mm_D3.2mm_P12.70mm_Horizontal
- U1: renamed from X1; value TFT680 -> 5MHz XTAL; footprint Crystal:Crystal_AT310_D3.0mm_L10.0mm_Horizontal -> Package_DIP:DIP-14_W7.62mm
- U2, U3: footprint (none) -> Package_DIP:DIP-14_W7.62mm
- U3: renamed from U2; footprint (none) -> Package_DIP:DIP-14_W7.62mm
- U4, U5: footprint (none) -> Package_DIP:DIP-16_W7.62mm
Connections:
- net +5V: now also U3.14 (VCC), U4.16 (VCC), U5.16 (VCC), C1.2, C2.2, C3.2, C4.2, C5.2, C6.2, C7.1, J1.11 (+5V), J2.21 (+5V), J2.23 (+5V), J2.25 (+5V)
- net GND: now also U3.7 (GND), U5.8 (GND), C1.1, C2.1, C3.1, C4.1, C5.1, C6.1, C7.2, J1.1 (GND), J1.3 (GND), J1.5 (GND), J1.7 (GND), J2.11 (GND), J2.13 (GND), J2.15 (GND), J2.9 (GND)
- net at U2.6 (~{Q}): now also J1.20 (PWM)
- net at U6.1 (A): now also U6.2 (B), J1.2 (CA0), J2.2 (PH0)
- net at U6.8 (CLK): now also J2.22 (MOTRCLK)
- new net: J1.18 (WRTDATA), J2.10 (WR)
- new net: J1.10 (WRTGATE), J2.12 (/WREQ)
- new net: J1.16 (RD), J2.14 (RD), J2.20 (SENSE)
- new net: J1.14 (ENBL), J2.16 (/DRVSEL)
- new net: J1.12 (SEL), J2.18 (HEADSEL)
- new net: J1.4 (CA1), J2.4 (PH1)
- new net: J1.6 (CA2), J2.6 (PH2)
- new net: J1.8 (LSTRB), J2.8 (PH3)
- new net +12V: J1.13 (+12V), J1.15 (+12V), J1.17 (+12V), J1.19 (+12V), J2.1 (+12V), J2.3 (+12V), J2.5 (+12V), J2.7 (+12V)
- no-connect marks 4 -> 12
Other:
- moved on the sheet: U1, U3A, U3B, U5, U6

Commit message: final commit for rev 1.0
Parts:
- added unit 3 of U2
Connections:
- net +5V: now also U2.14 (VCC); no longer J2.25 (+5V)
- net GND: now also U2.7 (GND)
- no-connect marks 12 -> 13
Other:
- note added: "DECOUPLING CAPACITORS"
- note added: "POWER CONNECTIONS"
- note added: "UNUSED"
- title: (none) -> Lisa Lite Adaptor
- moved on the sheet: C1, C2, C3, C4, C5, C6, C7, J1, J2, R1, U1, U2A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
